File: rescuedox_right/rescuedox_right.sch (KiCad schematic (older format))
At the start: 84 parts, among them SW110 SW_Push_45deg, SW111 SW_Push_45deg, SW112 SW_Push_45deg, SW113 SW_Push_45deg, SW114 SW_Push_45deg, SW115 SW_Push_45deg, SW116 SW_Push_45deg, SW18 SW_Push_45deg, SW19 SW_Push_45deg, SW210 SW_Push_45deg, SW211 SW_Push_45deg, SW212 SW_Push_45deg, SW213 SW_Push_45deg, SW214 SW_Push_45deg, SW215 SW_Push_45deg, SW216 SW_Push_45deg, SW28 SW_Push_45deg, SW29 SW_Push_45deg, SW310 SW_Push_45deg, SW311 SW_Push_45deg, SW312 SW_Push_45deg, SW313 SW_Push_45deg, SW314 SW_Push_45deg, SW315 SW_Push_45deg, SW316 SW_Push_45deg, SW38 SW_Push_45deg, SW39 SW_Push_45deg, SW410 SW_Push_45deg, SW411 SW_Push_45deg, SW412 SW_Push_45deg, SW413 SW_Push_45deg, SW415 SW_Push_45deg, SW48 SW_Push_45deg, SW49 SW_Push_45deg, SW510 SW_Push_45deg, SW511 SW_Push_45deg, SW512 SW_Push_45deg, SW514 SW_Push_45deg, SW515 SW_Push_45deg, SW516 SW_Push_45deg, SW58 SW_Push_45deg, SW59 SW_Push_45deg

Commit message: KiCad really doesn't like multiple boards in one project...
Parts:
- SW110, SW111, SW112, SW113, SW114, SW115, SW116, SW18, SW19, SW210, SW211, SW212, SW213, SW214, SW215, SW216, SW28, SW29, SW310, SW311, SW312, SW313, SW314, SW315, SW316, SW38, SW39, SW410, SW411, SW412, SW413, SW415, SW48, SW49, SW510, SW511, SW512, SW514, SW515, SW516, SW58, SW59: footprint (none) -> rescuedox:PG151101S11; Manufacturer Name (none) -> Kaihua Electronics; Manufacturer Part Number (none) -> PG151101S11
